File: PCB_TFG/tfg.brd (EAGLE design)
At the start: 85.1 x 58.4 mm, 11 parts

Commit message: final PCB
Parts:
- removed MSP430G2553_B: (no value), con-lsta:FE10
- MSP430G2553: device con-lsta:FE10 -> TI_MSP430_v16:N20
- moved MSP430G2553 7.73 mm to (30.5, 43.2)
Connections:
- net GND: now also MSP430G2553.20; no longer MSP430G2553_B.1
- net RST: now also MSP430G2553.16; no longer MSP430G2553_B.5
- net SCL: now also MSP430G2553.14; no longer MSP430G2553_B.7
- net SDA: now also MSP430G2553.15; no longer MSP430G2553_B.6
Routing:
- net LEN: track 62.3 -> 74.1 mm
- net V_VCC: track 152.0 -> 160.7 mm
- net GND: track 220.7 -> 214.9 mm, vias 6 -> 5
- net DN: track 33.1 -> 37.9 mm
- net SCLK: track 31.1 -> 35.9 mm
- net SDC: track 38.3 -> 41.3 mm
- net RST: track 80.2 -> 83.2 mm
- net S$3: track 39.0 -> 36.4 mm
- net SDA: track 46.8 -> 49.3 mm
- net SCL: track 49.8 -> 52.3 mm
- net SCE: track 48.7 -> 46.6 mm
